File: RepeatGame.sch (KiCad schematic (older format))
At the start: 27 parts, among them J1 BATTERY, J2 AVR-ISP-6, SW1 YELLOW, SW2 BLUE, SW3 ORANGE, SW4 RED, SW5 POWER, U1 ATmega328P-AU, Y1 12MHz

Commit message: Added source
Parts:
- R4, R6, R7: value 220 -> 330
- R5: value 100 -> 330
Changed lines of the file:
@@
 P 2000 4600
 F 0 "R4" H 2059 4646 50  0000 L CNN
-F 1 "220" H 2059 4555 50  0000 L CNN
+F 1 "330" H 2059 4555 50  0000 L CNN
 F 2 "Resistor_SMD:R_0805_2012Metric_Pad1.15x1.40mm_HandSolder" H 2000 4600 50  0001 C CNN
 F 3 "~" H 2000 4600 50  0001 C CNN
@@
 P 2500 4600
 F 0 "R5" H 2559 4646 50  0000 L CNN
-F 1 "100" H 2559 4555 50  0000 L CNN
+F 1 "330" H 2559 4555 50  0000 L CNN
 F 2 "Resistor_SMD:R_0805_2012Metric_Pad1.15x1.40mm_HandSolder" H 2500 4600 50  0001 C CNN
 F 3 "~" H 2500 4600 50  0001 C CNN
@@
 P 3000 4600
 F 0 "R6" H 3059 4646 50  0000 L CNN
-F 1 "220" H 3059 4555 50  0000 L CNN
+F 1 "330" H 3059 4555 50  0000 L CNN
 F 2 "Resistor_SMD:R_0805_2012Metric_Pad1.15x1.40mm_HandSolder" H 3000 4600 50  0001 C CNN
 F 3 "~" H 3000 4600 50  0001 C CNN
@@
 P 3500 4600
 F 0 "R7" H 3559 4646 50  0000 L CNN
-F 1 "220" H 3559 4555 50  0000 L CNN
+F 1 "330" H 3559 4555 50  0000 L CNN
 F 2 "Resistor_SMD:R_0805_2012Metric_Pad1.15x1.40mm_HandSolder" H 3500 4600 50  0001 C CNN
 F 3 "~" H 3500 4600 50  0001 C CNN
